Commit message: Update workspace to ROS 2 Jazzy and integrate Gazebo Harmonic with MoveIt 2

File: src/rover_arm_urdf/urdf/rover_arm_urdf.urdf (robot description, URDF)
Before this commit: robot rover_arm_urdf, 8 links, 7 joints
Links:
- added link world
Joints:
- added joint fixed_to_ground: type fixed, parent world, child base_link, origin xyz=0 0 0 rpy=0 0 0

Commit message: IK with fable

File: src/rover_arm_urdf/urdf/rover_arm_urdf.urdf (robot description, URDF)
Before this commit: robot rover_arm_urdf, 9 links, 8 joints
Links:
- added link tool_tip
- added link wrist_camera_link, mass 0.03; visual box size=0.03 0.06 0.02
- added link wrist_camera_optical_frame
Joints:
- added joint tool_tip_joint: type fixed, parent link_5_gripper_base, child tool_tip, origin xyz=0 0 0.123 rpy=0 0 0
- added joint wrist_camera_joint: type fixed, parent link_4_wrist_pitch_block, child wrist_camera_link, origin xyz=0.06 0 0.015 rpy=0 -1.5708 0
- added joint wrist_camera_optical_joint: type fixed, parent wrist_camera_link, child wrist_camera_optical_frame, origin xyz=0 0 0 rpy=-1.5708 0 -1.5708

Commit message: Update URDF configuration

File: src/rover_arm_urdf/urdf/rover_arm_urdf.urdf (robot description, URDF)
Before this commit: robot rover_arm_urdf, 9 links, 8 joints
Links:
- link link_6_left_jaw: geometry collision mesh filename=package://rover_arm_urdf/meshes/link_6_left_jaw.STL scale=1 2 4; visual mesh filename=package://rover_arm_urdf/meshes/link_6_left_jaw.STL scale=1 2 4
- link link_7_right_jaw: geometry collision mesh filename=package://rover_arm_urdf/meshes/link_7_right_jaw.STL scale=1 2 4; visual mesh filename=package://rover_arm_urdf/meshes/link_7_right_jaw.STL scale=1 2 4

Commit message: Updated URDF meshes, generated MoveIt 2 configuration, and added workspace visualization scripts

File: src/rover_arm_urdf/urdf/rover_arm_urdf.urdf (robot description, URDF)
Before this commit: robot rover_arm_urdf, 9 links, 8 joints
Links:
- link base_link: mass 2.2 -> 1.7
- link link_1_shoulder: mass 1.45 -> 0.85
- link link_2_upper_arm: mass 1.8 -> 1.25
- link link_3_forearm: mass 1.4 -> 1.1
- link link_4_wrist_pitch_block: mass 0.185 -> 0.15
- link link_5_gripper_base: mass 0.645 -> 0.5
- link link_6_left_jaw: mass 0.03 -> 0.1; geometry collision mesh filename=package://rover_arm_urdf/meshes/link_6_left_jaw.STL; visual mesh filename=package://rover_arm_urdf/meshes/link_6_left_jaw.STL
- link link_7_right_jaw: mass 0.03 -> 0.1; geometry collision mesh filename=package://rover_arm_urdf/meshes/link_7_right_jaw.STL; visual mesh filename=package://rover_arm_urdf/meshes/link_7_right_jaw.STL
Joints:
- joint joint_1_base_roll: axis 0 0 1 -> 0 0 -1; limit lower=0 upper=0 effort=30 velocity=7.33 -> lower=-1.57 upper=1.57 effort=30 velocity=7.33; type continuous -> revolute
- joint joint_2_shoulder_pitch: limit lower=0 upper=1.57 effort=30 velocity=7.33 -> lower=0 upper=2.88 effort=30 velocity=7.33; origin xyz=0 0 0.0875 rpy=0 0 0 -> xyz=0 -0.0075 0.095 rpy=0 -1.309 0
- joint joint_3_elbow_pitch: limit lower=0 upper=1.57 effort=30 velocity=7.33 -> lower=-2.88 upper=0 effort=30 velocity=7.33; origin xyz=0 0 0.4725 rpy=0 0 0 -> xyz=0 0.1205 0.4725 rpy=3.1416 0.2618 3.1416
- joint joint_4_wrist_pitch: limit lower=0 upper=1.57 effort=8.5 velocity=9 -> lower=-1.57 upper=1.57 effort=8.5 velocity=9
- joint joint_5_wrist_roll: limit effort=8.5 velocity=9 -> lower=-3.142 upper=3.142 effort=8.5 velocity=9; origin xyz=0 0 0.03 rpy=0 0 0 -> xyz=0 0 0.09675 rpy=0 0 0; type continuous -> revolute
- joint joint_6_left_jaw: limit lower=0 upper=0.08 effort=60 velocity=0.1 -> lower=0 upper=0.045 effort=50 velocity=0.1; origin xyz=0 0 0.07325 rpy=0 0 0 -> xyz=0 0.016961 0.05375 rpy=0 0 0
- joint joint_7_right_jaw: limit lower=-0.08 upper=0 effort=60 velocity=0.1 -> lower=0 upper=0.045 effort=50 velocity=0.1; origin xyz=0 0 0.07325 rpy=0 0 0 -> xyz=0 -0.016961 0.05375 rpy=0 0 0
